Commit message: Add files via upload

File: Pydrake Model/models/HexRotor.urdf.xacro (robot description, xacro)
@@ -62,4 +62,6 @@
   <xacro:property name="prop_joint_origin_r" value = "${split_xsize/2} ${-split_ysize/2} ${split_zsize/2}"/>
   <xacro:property name="prop_joint_origin_l" value = "${-split_xsize/2} ${-split_ysize/2} ${split_zsize/2}"/>
+  <!-- <xacro:property name="prop_joint_origin_r" value = "${split_xsize/2} 0.0 ${split_zsize/2}"/> -->
+  <!-- <xacro:property name="prop_joint_origin_l" value = "${-split_xsize/2} 0.0 ${split_zsize/2}"/> -->
   <xacro:property name="prop_joint_rpy" value = "${pi/2} 0.0 0.0"/>
   <!-- #endregion -->
@@ -350,5 +352,6 @@
     <parent link="rotor_base"/>
     <child link="rotor_arm_1"/>
-    <origin xyz="0.0 ${base_radius} 0.0" rpy="${-pi/2} 0.0 0.0"/>
+    <!-- <origin xyz="${base_radius*cos(pi/6)} ${-base_radius*sin(pi/6)} 0.0" rpy="${-pi/2} 0.0 ${-pi/6-pi/2}"/> -->
+    <origin xyz="${base_radius*sin(pi/6)} ${base_radius*cos(pi/6)} 0.0" rpy="${-pi/2} 0.0 ${-pi/6}"/>
     <axis xyz="${arm_joint_axis}"/>
     <limit lower="${-arm_joint_limit}" upper="${arm_joint_limit}" effort="${arm_joint_effort}" velocity="1.0"/>
@@ -357,5 +360,6 @@
     <parent link="rotor_base"/>
     <child link="rotor_arm_2"/>
-    <origin xyz="${base_radius*cos(pi/6)} ${-base_radius*sin(pi/6)} 0.0" rpy="${-pi/2} 0.0 ${-pi/6-pi/2}"/>
+    <!-- <origin xyz="0.0 ${base_radius} 0.0" rpy="${-pi/2} 0.0 0.0"/> -->
+    <origin xyz="${-base_radius} 0.0 0.0" rpy="${-pi/2} 0.0 ${pi/2}"/>
     <axis xyz="${arm_joint_axis}"/>
     <limit lower="${-arm_joint_limit}" upper="${arm_joint_limit}" effort="${arm_joint_effort}" velocity="1.0"/>
@@ -364,5 +368,6 @@
     <parent link="rotor_base"/>
     <child link="rotor_arm_3"/>
-    <origin xyz="${-base_radius*cos(pi/6)} ${-base_radius*sin(pi/6)} 0.0" rpy="${-pi/2} 0.0 ${+pi/6+pi/2}"/>
+    <!-- <origin xyz="${-base_radius*cos(pi/6)} ${-base_radius*sin(pi/6)} 0.0" rpy="${-pi/2} 0.0 ${+pi/6+pi/2}"/> -->
+    <origin xyz="${base_radius*sin(pi/6)} ${-base_radius*cos(pi/6)} 0.0" rpy="${-pi/2} 0.0 ${-pi/6-2*pi/3}"/>
     <axis xyz="${arm_joint_axis}"/>
     <limit lower="${-arm_joint_limit}" upper="${arm_joint_limit}" effort="${arm_joint_effort}" velocity="1.0"/>

Commit message: Add files via upload

File: Pydrake Model/models/HexRotor.urdf.xacro (robot description, xacro)
@@ -9,60 +9,69 @@
   <!-- TO DO
     - update dimensions
+    - utilize xacro capabilities/macros to automate file generation
+    - implement more file arguments for parsing
+    - use .yaml for config?
     -
   -->
+  <!-- #region Xacro Arguments -->
+  <xacro:arg name="base_radius_arg" default="0.0"/>
+  <xacro:arg name="arm_radius_arg" default="0.0"/>
+  <xacro:arg name="arm_length_arg" default="0.0"/>
+  <xacro:arg name="split_zsize_arg" default="0.0"/>
+  <!-- #endregion -->
   <!-- #region Xacro Definitions -->
   <xacro:property name="pi" value="3.141592653589793"/>
-  <xacro:property name="zero_origin" value = "0.0 0.0 0.0"/>
-  <xacro:property name="zero_rpy" value = "0.0 0.0 0.0"/>
-  <xacro:property name="base_radius" value = "${0.15/2}"/>
-  <xacro:property name="base_length" value = "0.05"/>
-  <xacro:property name="base_origin" value = "${zero_origin}"/>
-  <xacro:property name="base_mass" value = "0.5"/>
-  <xacro:property name="base_ixx" value = "${(base_mass*base_radius**2)/4 + (base_mass*base_length**2)/12}"/>
-  <xacro:property name="base_iyy" value = "${(base_mass*base_radius**2)/4 + (base_mass*base_length**2)/12}"/>
-  <xacro:property name="base_izz" value = "${(base_mass*base_radius**2)/2}"/>
-  <xacro:property name="base_ixy" value = "0.0"/>
-  <xacro:property name="base_ixz" value = "0.0"/>
-  <xacro:property name="base_iyz" value = "0.0"/>
-  <xacro:property name="arm_radius" value = "0.02"/>
-  <xacro:property name="arm_length" value = "0.1"/>
-  <xacro:property name="arm_origin" value = "0.0 0.0 ${arm_length/2}"/>
-  <xacro:property name="arm_mass" value = "0.05"/>
-  <xacro:property name="arm_ixx" value = "${(arm_mass*arm_radius**2)/4 + (arm_mass*arm_length**2)/3}"/>
-  <xacro:property name="arm_iyy" value = "${(arm_mass*arm_radius**2)/4 + (arm_mass*arm_length**2)/3}"/>
-  <xacro:property name="arm_izz" value = "${(arm_mass*arm_radius**2)/2}"/>
-  <xacro:property name="arm_ixy" value = "0.0"/>
-  <xacro:property name="arm_ixz" value = "0.0"/>
-  <xacro:property name="arm_iyz" value = "0.0"/>
-  <xacro:property name="arm_joint_axis" value = "0.0 0.0 1.0"/>
-  <xacro:property name="arm_joint_limit" value = "${4*pi}"/>
-  <xacro:property name="arm_joint_effort" value = "0.0"/>
-  <xacro:property name="split_xsize" value = "0.2"/>
-  <xacro:property name="split_ysize" value = "${2*arm_radius}"/>
-  <xacro:property name="split_zsize" value = "0.05"/>
-  <xacro:property name="split_origin" value = "0.0 0.0 ${split_zsize/2}"/>
-  <xacro:property name="split_mass" value = "0.1"/>
-  <xacro:property name="split_ixx" value = "${(split_mass*(split_ysize**2+split_zsize**2))/12 + split_mass*(split_zsize/2)**2}"/>
-  <xacro:property name="split_iyy" value = "${(split_mass*(split_xsize**2+split_zsize**2))/12 + split_mass*(split_zsize/2)**2}"/>
-  <xacro:property name="split_izz" value = "${(split_mass*(split_xsize**2+split_ysize**2))/12}"/>
-  <xacro:property name="split_ixy" value = "0.0"/>
-  <xacro:property name="split_ixz" value = "0.0"/>
-  <xacro:property name="split_iyz" value = "0.0"/>
-  <xacro:property name="split_joint_origin" value = "0.0 0.0 ${arm_length}"/>
-  <xacro:property name="prop_radius" value = "0.06"/>
-  <xacro:property name="prop_length" value = "0.01"/>
-  <xacro:property name="prop_origin" value = "0.0 0.0 ${prop_length/2}"/>
-  <xacro:property name="prop_mass" value = "0.001"/>
-  <xacro:property name="prop_ixx" value = "${(prop_mass*prop_radius**2)/4 + (prop_mass*prop_length**2)/12}"/>
-  <xacro:property name="prop_iyy" value = "${(prop_mass*prop_radius**2)/4 + (prop_mass*prop_length**2)/12}"/>
-  <xacro:property name="prop_izz" value = "${(prop_mass*prop_radius**2)/2}"/>
-  <xacro:property name="prop_ixy" value = "0.0"/>
-  <xacro:property name="prop_ixz" value = "0.0"/>
-  <xacro:property name="prop_iyz" value = "0.0"/>
-  <xacro:property name="prop_joint_origin_r" value = "${split_xsize/2} ${-split_ysize/2} ${split_zsize/2}"/>
-  <xacro:property name="prop_joint_origin_l" value = "${-split_xsize/2} ${-split_ysize/2} ${split_zsize/2}"/>
-  <!-- <xacro:property name="prop_joint_origin_r" value = "${split_xsize/2} 0.0 ${split_zsize/2}"/> -->
-  <!-- <xacro:property name="prop_joint_origin_l" value = "${-split_xsize/2} 0.0 ${split_zsize/2}"/> -->
-  <xacro:property name="prop_joint_rpy" value = "${pi/2} 0.0 0.0"/>
+  <xacro:property name="zero_origin" value="0.0 0.0 0.0"/>
+  <xacro:property name="zero_rpy" value="0.0 0.0 0.0"/>
+  <xacro:property name="base_radius" value="$(arg base_radius_arg)"/>
+  <xacro:property name="base_length" value="0.05"/>
+  <xacro:property name="base_origin" value="${zero_origin}"/>
+  <xacro:property name="base_mass" value="0.5"/>
+  <xacro:property name="base_ixx" value="${(base_mass*base_radius**2)/4 + (base_mass*base_length**2)/12}"/>
+  <xacro:property name="base_iyy" value="${(base_mass*base_radius**2)/4 + (base_mass*base_length**2)/12}"/>
+  <xacro:property name="base_izz" value="${(base_mass*base_radius**2)/2}"/>
+  <xacro:property name="base_ixy" value="0.0"/>
+  <xacro:property name="base_ixz" value="0.0"/>
+  <xacro:property name="base_iyz" value="0.0"/>
+  <xacro:property name="arm_radius" value="$(arg arm_radius_arg)"/>
+  <xacro:property name="arm_length" value="$(arg arm_length_arg)"/>
+  <xacro:property name="arm_origin" value="0.0 0.0 ${arm_length/2}"/>
+  <xacro:property name="arm_mass" value="0.05"/>
+  <xacro:property name="arm_ixx" value="${(arm_mass*arm_radius**2)/4 + (arm_mass*arm_length**2)/3}"/>
+  <xacro:property name="arm_iyy" value="${(arm_mass*arm_radius**2)/4 + (arm_mass*arm_length**2)/3}"/>
+  <xacro:property name="arm_izz" value="${(arm_mass*arm_radius**2)/2}"/>
+  <xacro:property name="arm_ixy" value="0.0"/>
+  <xacro:property name="arm_ixz" value="0.0"/>
+  <xacro:property name="arm_iyz" value="0.0"/>
+  <xacro:property name="arm_joint_axis" value="0.0 0.0 1.0"/>
+  <xacro:property name="arm_joint_limit" value="${4*pi}"/>
+  <xacro:property name="arm_joint_effort" value="0.0"/>
+  <xacro:property name="split_xsize" value="0.2"/>
+  <xacro:property name="split_ysize" value="${2*arm_radius}"/>
+  <xacro:property name="split_zsize" value="$(arg split_zsize_arg)"/>
+  <xacro:property name="split_origin" value="0.0 0.0 ${split_zsize/2}"/>
+  <xacro:property name="split_mass" value="0.1"/>
+  <xacro:property name="split_ixx" value="${(split_mass*(split_ysize**2+split_zsize**2))/12 + split_mass*(split_zsize/2)**2}"/>
+  <xacro:property name="split_iyy" value="${(split_mass*(split_xsize**2+split_zsize**2))/12 + split_mass*(split_zsize/2)**2}"/>
+  <xacro:property name="split_izz" value="${(split_mass*(split_xsize**2+split_ysize**2))/12}"/>
+  <xacro:property name="split_ixy" value="0.0"/>
+  <xacro:property name="split_ixz" value="0.0"/>
+  <xacro:property name="split_iyz" value="0.0"/>
+  <xacro:property name="split_joint_origin" value="0.0 0.0 ${arm_length}"/>
+  <xacro:property name="prop_radius" value="0.06"/>
+  <xacro:property name="prop_length" value="0.01"/>
+  <xacro:property name="prop_origin" value="0.0 0.0 ${prop_length/2}"/>
+  <xacro:property name="prop_mass" value="0.001"/>
+  <xacro:property name="prop_ixx" value="${(prop_mass*prop_radius**2)/4 + (prop_mass*prop_length**2)/12}"/>
+  <xacro:property name="prop_iyy" value="${(prop_mass*prop_radius**2)/4 + (prop_mass*prop_length**2)/12}"/>
+  <xacro:property name="prop_izz" value="${(prop_mass*prop_radius**2)/2}"/>
+  <xacro:property name="prop_ixy" value="0.0"/>
+  <xacro:property name="prop_ixz" value="0.0"/>
+  <xacro:property name="prop_iyz" value="0.0"/>
+  <xacro:property name="prop_joint_origin_r" value="${split_xsize/2} ${-split_ysize/2} ${split_zsize/2}"/>
+  <xacro:property name="prop_joint_origin_l" value="${-split_xsize/2} ${-split_ysize/2} ${split_zsize/2}"/>
+  <!-- <xacro:property name="prop_joint_origin_r" value="${split_xsize/2} 0.0 ${split_zsize/2}"/> -->
+  <!-- <xacro:property name="prop_joint_origin_l" value="${-split_xsize/2} 0.0 ${split_zsize/2}"/> -->
+  <xacro:property name="prop_joint_rpy" value="${pi/2} 0.0 0.0"/>
   <!-- #endregion -->
   <!-- #region Material Definitions -->
